File: hardware/ESP32-C3-DevKitM-1.kicad_sch (KiCad schematic)
At the start: 0 parts

Commit message: Hardware: Updated Schematics and inicial ESP32 schematic
Parts:
- added C1: 100nf, symbol Device:C
- added SW1: SW_Push_RST, symbol Switch:SW_Push
- added U1: ESP32-C3-DevKitM-1, RF_Module:ESP32-C3-DevKitM-1, symbol RF_Module:ESP32-C3-DevKitM-1
Connections:
- new net 3,3V: U1.2 (3V3), U1.3 (3V3)
- new net 5V: U1.13 (5V), U1.14 (5V)
- new net CS (LOAD): U1.11 (IO10)
- new net GND: C1.1, SW1.1, U1.1 (GND), U1.12 (GND), U1.15 (GND), U1.16 (GND), U1.19 (GND), U1.24 (GND), U1.27 (GND), U1.30 (GND), U1.6 (GND), U1.8 (GND)
- new net I2C SCL: U1.21 (IO5)
- new net I2C SDA: U1.20 (IO4)
- new net MOSI (DIN): U1.22 (IO6)
- new net RST: C1.2, SW1.2, U1.7 (RST)
- new net SCK (CLK): U1.23 (IO7)
- new net USB Data Minus: U1.18 (IO18)
- new net USB Data Plus: U1.17 (IO19)
- no-connect marks 0 -> 3
Other:
- note added: "ESP32-C3-DevKitM-1"
- note added: "EXTERNAL CONNECTIONS"
- note added: "I2C"
- note added: "POWER"
- note added: "RESET BOTTON"
- note added: "SPI"
- note added: "USB"
